File: KiCad/numpad/KITTEN.kicad_sch (KiCad schematic)
At the start: 46 parts, among them J1 Barrel_Jack_Switch, J10 Conn_01x02_Pin, J2 Conn_01x03_Pin, J3 Conn_01x04_Pin, J4 Conn_01x05_Pin, J5 Conn_01x06_Pin, J6 Conn_01x07_Pin, J7 Conn_01x08_Pin, J8 Conn_01x09_Pin, J9 Conn_01x10_Pin, SW1 Cherry Switch Single, SW10 Cherry Switch Single, SW11 Cherry Switch Single, SW12 Cherry Switch Single, SW13 Cherry Switch Single, SW2 Cherry Switch 1.5x - Enter Key, SW3 Cherry Switch Single, SW4 Cherry Switch Single, SW5 Cherry Switch Single, SW6 Cherry Switch Single, SW7 Cherry Switch Single, SW9 Cherry Switch Single, U2 TMC2209, U3 Display, U4 ICM-20948, U5 24LC512, U6 Adafruit_ICM20948, U7 LTV-817S, U8 TL431D, U9 LT1632

Commit message: Display and numpad schematics
Parts:
- removed J1: Barrel_Jack_Switch, Connector_BarrelJack:BarrelJack_Wuerth_694106106102_2.0x5.5mm, symbol Connector:Barrel_Jack_Switch
- removed J10: Conn_01x02_Pin, Connector_JST:JST_PH_B2B-PH-K_1x02_P2.00mm_Vertical, symbol Connector:Conn_01x02_Pin
- removed J2: Conn_01x03_Pin, Connector_JST:JST_PH_B3B-PH-K_1x03_P2.00mm_Vertical, symbol Connector:Conn_01x03_Pin
- removed J3: Conn_01x04_Pin, Connector_JST:JST_PH_B4B-PH-K_1x04_P2.00mm_Vertical, symbol Connector:Conn_01x04_Pin
- removed J4: Conn_01x05_Pin, Connector_JST:JST_PH_B5B-PH-K_1x05_P2.00mm_Vertical, symbol Connector:Conn_01x05_Pin
- removed J5: Conn_01x06_Pin, Connector_JST:JST_PH_B6B-PH-K_1x06_P2.00mm_Vertical, symbol Connector:Conn_01x06_Pin
- removed J6: Conn_01x07_Pin, Connector_JST:JST_PH_B7B-PH-K_1x07_P2.00mm_Vertical, symbol Connector:Conn_01x07_Pin
- removed J7: Conn_01x08_Pin, Connector_JST:JST_PH_B8B-PH-K_1x08_P2.00mm_Vertical, symbol Connector:Conn_01x08_Pin
- removed J8: Conn_01x09_Pin, Connector_JST:JST_PH_B9B-PH-K_1x09_P2.00mm_Vertical, symbol Connector:Conn_01x09_Pin
- removed J9: Conn_01x10_Pin, Connector_JST:JST_PH_B10B-PH-K_1x10_P2.00mm_Vertical, symbol Connector:Conn_01x10_Pin
- removed SW1: Cherry Switch Single, ComponentLib:SW_Cherry_MX_1.00u_PCB, symbol Switch:SW_Push
- removed SW2: Cherry Switch 1.5x - Enter Key, ComponentLib:SW_Cherry_MX_1.50u_PCB, symbol Switch:SW_Push
- removed U1: ~, ComponentLib:NUCLEO-F767ZI, symbol SymbolLib:NUCLEO-F767ZI
- removed U2: TMC2209, ComponentLib:TMC2209 Silentstepstick, symbol SymbolLib:TMC2209_Silentstepstick
- removed U3: Display, ComponentLib:NHD-2.23-12832UCB3, symbol SymbolLib:NHD-2.23-12832UCB3
- removed U4: ICM-20948, ComponentLib:ICM-20948, symbol Sensor_Motion:ICM-20948
- removed U5: 24LC512, Package_SO:SOIC-8_5.3x6.2mm_P1.27mm, symbol Memory_EEPROM:24LC512
- removed U6: Adafruit_ICM20948, ComponentLib:Adafruit-ICM-20948, symbol SymbolLib:Adafruit_ICM20948
- removed U7: LTV-817S, Package_DIP:SMDIP-4_W9.53mm, symbol Isolator:LTV-817S
- added C1, C3: C, Capacitor_SMD:C_0603_1608Metric_Pad1.08x0.95mm_HandSolder, symbol Device:C
- added C2: 1n, Capacitor_SMD:C_0603_1608Metric, symbol Device:C
- added D1: LED, symbol Device:LED
- added J12: Conn_01x04_Pin, Connector_JST:JST_PH_B4B-PH-K_1x04_P2.00mm_Vertical, symbol Connector:Conn_01x04_Pin
- added R16, R19: 0R, Resistor_SMD:R_0603_1608Metric, symbol Device:R
- added R17, R20: 100R, Resistor_SMD:R_0603_1608Metric, symbol Device:R
- added R18: 1k, Resistor_SMD:R_0603_1608Metric, symbol Device:R
- added R21: 330R, Resistor_SMD:R_0603_1608Metric, symbol Device:R
- added TP1, TP2: TestPoint, TestPoint:TestPoint_Pad_D2.0mm, symbol Connector:TestPoint
- R1, R11, R12, R2, R3, R4, R5, R6, R7, R8, R9: value R -> 1k
- R10: value R -> 100k
- R13: value R -> 10k
- R14: value R -> 51k
- R15: value R -> 7k5
Connections:
- net V+ is gone; now on net +5V: U9.8 (V+)
- net V- is gone; now on net GND: U9.4 (V-)
- net GND: now also R14.2, R15.2, U8.2 (A), U8.3 (A), U8.6 (A), U8.7 (A), C1.2, C2.2, C3.2, D1.1 (K), J12.4 (Pin_4)
- net at R10.1, SW10.2, SW11.2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: now also R18.1
- net 3Vref: now reaches R15.1
- net 3Vref: now also R1.1, R12.2, R13.1, SW3.1, U8.1 (K), U9.3 (A+), TP1.1
- net +5V: now reaches R12.1
- net +5V: now also J12.1 (Pin_1), R21.1
- net NumpadOut: now reaches U9.5 (B+)
- net NumpadOut: now also C2.1, R18.2, TP2.1
- net at U9.6 (B-): now also C3.1, R19.1
- net at U9.7 (OUT_B): now also R19.2, R20.1
- net at U8.8 (REF): now also R13.2, R14.1
- net at U9.1 (OUT_A): now also R16.2, R17.1
- net at U9.2 (A-): now also C1.1, R16.1
- new net: D1.2 (A), R21.2
- new net NumpadOut_toADC: J12.3 (Pin_3), R20.2
- new net VREF_measback: J12.2 (Pin_2), R17.2
Other:
- note added: "Csatlakozó"
- note added: "Numpad"
- note added: "Numpadkimenet visszamérése"
- note added: "Opamp tápellátás"
- note added: "Referenciafeszültség előállítása"
- note added: "Referenciafeszültség visszamérése"
- note added: "V_{out} = 2.5V×(1+R_{1}/R_{2})"
- note added: "Visszajelző LED"
- moved on the sheet: R1, R10, R11, R12, R13, R14, R15, R2, R3, R4, R5, R6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
