File: KiCad/motherboard/motherboard.kicad_pcb (KiCad board)
At the start: 2 copper layers, 19 parts, among them J1 Barrel_Jack_Switch, J10 Conn_01x02_Pin, J2 Conn_01x03_Pin, J3 Conn_01x04_Pin, J4 Conn_01x05_Pin, J5 Conn_01x06_Pin, J6 Conn_01x07_Pin, J7 Conn_01x08_Pin, J8 Conn_01x09_Pin, J9 Conn_01x10_Pin, SW1 Cherry Switch Single, SW2 Cherry Switch 1.5x - Enter Key, U2 TMC2209, U3 Display, U4 ICM-20948, U5 24LC512, U6 Adafruit_ICM20948, U7 LTV-817S

Commit message: main board pcb design started
Parts:
- removed J10: Conn_01x02_Pin, Connector_JST:JST_PH_B2B-PH-K_1x02_P2.00mm_Vertical
- removed J9: Conn_01x10_Pin, Connector_JST:JST_PH_B10B-PH-K_1x10_P2.00mm_Vertical
- removed SW1: Cherry Switch Single, ComponentLib:SW_Cherry_MX_1.00u_PCB
- removed SW2: Cherry Switch 1.5x - Enter Key, ComponentLib:SW_Cherry_MX_1.50u_PCB
- added C1: 100n, Capacitor_SMD:C_0603_1608Metric, F.Cu at (72.3, 64.1)
- added C18: 100n, Capacitor_SMD:C_0603_1608Metric, F.Cu at (243.2, 92.5)
- added C19: 100n, Capacitor_SMD:C_0603_1608Metric, F.Cu at (250.8, 92.5)
- added C2: 22u, 35V, Capacitor_SMD:C_1206_3216Metric, F.Cu at (179.6, 96.1)
- added C20: 100n, Capacitor_SMD:C_0603_1608Metric, F.Cu at (258.4, 92.5)
- added C21: 100n, Capacitor_SMD:C_0603_1608Metric, F.Cu at (266.0, 92.5)
- added C3: 22u, 35V, Capacitor_SMD:C_1206_3216Metric, F.Cu at (184.6, 96.1)
- added C4: 22u, 35V, Capacitor_SMD:C_1206_3216Metric, F.Cu at (206.1, 96.4)
- added C5: 22u, 35V, Capacitor_SMD:C_1206_3216Metric, F.Cu at (211.1, 96.4)
- added C6: 1u, Capacitor_SMD:C_0603_1608Metric, F.Cu at (43.3, 154.8)
- added C7: 1u, Capacitor_SMD:C_0603_1608Metric, F.Cu at (75.3, 134.6)
- added C8: 100n, Capacitor_SMD:C_0603_1608Metric, F.Cu at (259.4, 21.6)
- added C9: 1u, Capacitor_SMD:C_0603_1608Metric, F.Cu at (259.4, 19.7)
- added D1: RED_LED, Diode_SMD:D_0603_1608Metric, F.Cu at (94.2, 64.1)
- added D10: GREEN_LED, Diode_SMD:D_0603_1608Metric, F.Cu at (50.3, 140.0)
- added D11: GREEN_LED, Diode_SMD:D_0603_1608Metric, F.Cu at (68.3, 149.4)
- added D2: SZSMF6L24CAT3G, Diode_SMD:D_SOD-123, F.Cu at (233.7, 57.8)
- added D3: V8PAM103HM3H, Diode_SMD:Vishay_SMPA, F.Cu at (248.3, 48.2)
- added D4: GREEN_LED, Diode_SMD:D_0603_1608Metric, F.Cu at (238.8, 51.5)
- added D5: RED_LED, Diode_SMD:D_0603_1608Metric, F.Cu at (242.4, 51.5)
- added D6: GREEN_LED, Diode_SMD:D_0603_1608Metric, F.Cu at (255.0, 54.8)
- added D7: GREEN_LED, Diode_SMD:D_0603_1608Metric, F.Cu at (189.6, 91.1)
- added D8: GREEN_LED, Diode_SMD:D_0603_1608Metric, F.Cu at (216.2, 91.1)
- added D9: GREEN_LED, Diode_SMD:D_0603_1608Metric, F.Cu at (28.9, 173.6)
- added F1: 576-0154007.DRTL, Fuse:Fuseholder_Littelfuse_Nano2_154x, F.Cu at (230.7, 50.7)
- added J11: Conn_01x06_Pin, Connector_JST:JST_PH_B6B-PH-K_1x06_P2.00mm_Vertical, F.Cu at (22.1, 73.7)
- added J12: Conn_01x06_Pin, Connector_JST:JST_PH_B6B-PH-K_1x06_P2.00mm_Vertical, F.Cu at (22.1, 56.0)
- added J13: Conn_01x04_Pin, Connector_JST:JST_PH_B4B-PH-K_1x04_P2.00mm_Vertical, F.Cu at (22.2, 39.5)
- added J14: Conn_01x04_Pin, Connector_JST:JST_PH_B4B-PH-K_1x04_P2.00mm_Vertical, F.Cu at (221.7, 136.7)
- added J15: Conn_01x04_Pin, Connector_JST:JST_PH_B4B-PH-K_1x04_P2.00mm_Vertical, F.Cu at (268.3, 136.2)
- added J17: DB25_Socket_MountingHoles, Connector_Dsub:DSUB-25_Socket_Horizontal_P2.77x2.84mm_EdgePinOffset7.70mm_Housed_MountingHolesOffset9.12mm, F.Cu at (75.1, 174.5)
- added J18: Conn_01x09_Pin, Connector_JST:JST_PH_B9B-PH-K_1x09_P2.00mm_Vertical, F.Cu at (22.2, 110.8)
- added JP1: SolderJumper_2_Open, Jumper:SolderJumper-2_P1.3mm_Open_RoundedPad1.0x1.5mm, F.Cu at (181.3, 32.3)
- added JP10: SolderJumper_2_Open, Resistor_SMD:R_0603_1608Metric_Pad0.98x0.95mm_HandSolder, F.Cu at (-53.3, -134.6)
- added JP100: SolderJumper_2_Open, Resistor_SMD:R_0603_1608Metric_Pad0.98x0.95mm_HandSolder, F.Cu at (-109.7, 117.1)
- added JP101: SolderJumper_2_Open, Resistor_SMD:R_0603_1608Metric_Pad0.98x0.95mm_HandSolder, F.Cu at (-109.7, 119.6)
- added JP102: SolderJumper_2_Open, Resistor_SMD:R_0603_1608Metric_Pad0.98x0.95mm_HandSolder, F.Cu at (-109.7, 122.1)
- added JP103: SolderJumper_2_Open, Resistor_SMD:R_0603_1608Metric_Pad0.98x0.95mm_HandSolder, F.Cu at (-109.7, 124.6)
- added JP104: SolderJumper_2_Open, Resistor_SMD:R_0603_1608Metric_Pad0.98x0.95mm_HandSolder, F.Cu at (-109.7, 127.1)
- added JP105: SolderJumper_2_Open, Resistor_SMD:R_0603_1608Metric_Pad0.98x0.95mm_HandSolder, F.Cu at (-109.7, 129.7)
- added JP106: SolderJumper_2_Open, Resistor_SMD:R_0603_1608Metric_Pad0.98x0.95mm_HandSolder, F.Cu at (-109.7, 132.2)
- added JP107: SolderJumper_2_Open, Resistor_SMD:R_0603_1608Metric_Pad0.98x0.95mm_HandSolder, F.Cu at (-109.7, 134.7)
- added JP108: SolderJumper_2_Open, Resistor_SMD:R_0603_1608Metric_Pad0.98x0.95mm_HandSolder, F.Cu at (-109.7, 137.2)
- added JP109: SolderJumper_2_Open, Resistor_SMD:R_0603_1608Metric_Pad0.98x0.95mm_HandSolder, F.Cu at (-109.7, 139.7)
- added JP11: SolderJumper_2_Open, Resistor_SMD:R_0603_1608Metric_Pad0.98x0.95mm_HandSolder, F.Cu at (-53.3, -132.1)
- added JP110: SolderJumper_2_Open, Resistor_SMD:R_0603_1608Metric_Pad0.98x0.95mm_HandSolder, F.Cu at (-105.4, 109.6)
- added JP111: SolderJumper_2_Open, Resistor_SMD:R_0603_1608Metric_Pad0.98x0.95mm_HandSolder, F.Cu at (-105.4, 112.1)
- added JP112: SolderJumper_2_Open, Resistor_SMD:R_0603_1608Metric_Pad0.98x0.95mm_HandSolder, F.Cu at (-105.4, 114.6)
- added JP113: SolderJumper_2_Open, Resistor_SMD:R_0603_1608Metric_Pad0.98x0.95mm_HandSolder, F.Cu at (-105.4, 117.1)
- added JP114: SolderJumper_2_Open, Resistor_SMD:R_0603_1608Metric_Pad0.98x0.95mm_HandSolder, F.Cu at (-105.4, 119.6)
- added JP115: SolderJumper_2_Open, Resistor_SMD:R_0603_1608Metric_Pad0.98x0.95mm_HandSolder, F.Cu at (-105.4, 122.1)
- added JP116: SolderJumper_2_Open, Resistor_SMD:R_0603_1608Metric_Pad0.98x0.95mm_HandSolder, F.Cu at (-105.4, 124.6)
- added JP117: SolderJumper_2_Open, Resistor_SMD:R_0603_1608Metric_Pad0.98x0.95mm_HandSolder, F.Cu at (-105.4, 127.1)
- added JP118: SolderJumper_2_Open, Resistor_SMD:R_0603_1608Metric_Pad0.98x0.95mm_HandSolder, F.Cu at (-105.4, 129.7)
- added JP119: SolderJumper_2_Bridged, Resistor_SMD:R_0603_1608Metric, F.Cu at (79.8, 60.3)
- added JP12: SolderJumper_2_Open, Resistor_SMD:R_0603_1608Metric_Pad0.98x0.95mm_HandSolder, F.Cu at (-53.3, -129.5)
- added JP120: Jumper_2_Bridged, Connector_PinHeader_2.54mm:PinHeader_1x02_P2.54mm_Vertical, F.Cu at (144.8, 58.4)
- added JP121: SolderJumper_2_Open, Resistor_SMD:R_0603_1608Metric, F.Cu at (82.3, 60.3)
- added JP13: SolderJumper_2_Open, Resistor_SMD:R_0603_1608Metric_Pad0.98x0.95mm_HandSolder, F.Cu at (-53.3, -127.0)
- added JP14: SolderJumper_2_Open, Resistor_SMD:R_0603_1608Metric_Pad0.98x0.95mm_HandSolder, F.Cu at (-53.3, -124.5)
- added JP15: SolderJumper_2_Open, Resistor_SMD:R_0603_1608Metric_Pad0.98x0.95mm_HandSolder, F.Cu at (-53.3, -122.0)
- added JP16: SolderJumper_2_Open, Resistor_SMD:R_0603_1608Metric_Pad0.98x0.95mm_HandSolder, F.Cu at (-53.3, -119.5)
- added JP17: SolderJumper_2_Open, Resistor_SMD:R_0603_1608Metric_Pad0.98x0.95mm_HandSolder, F.Cu at (-53.3, -117.0)
- added JP18: SolderJumper_2_Open, Resistor_SMD:R_0603_1608Metric_Pad0.98x0.95mm_HandSolder, F.Cu at (-53.3, -114.5)
- added JP19: SolderJumper_2_Open, Resistor_SMD:R_0603_1608Metric_Pad0.98x0.95mm_HandSolder, F.Cu at (-49.0, -144.6)
- added JP2: SolderJumper_2_Open, Jumper:SolderJumper-2_P1.3mm_Open_RoundedPad1.0x1.5mm, F.Cu at (244.7, 22.9)
- added JP20: SolderJumper_2_Open, Resistor_SMD:R_0603_1608Metric_Pad0.98x0.95mm_HandSolder, F.Cu at (-49.0, -142.1)
- added JP21: SolderJumper_2_Open, Resistor_SMD:R_0603_1608Metric_Pad0.98x0.95mm_HandSolder, F.Cu at (-49.0, -139.6)
- added JP22: SolderJumper_2_Open, Resistor_SMD:R_0603_1608Metric_Pad0.98x0.95mm_HandSolder, F.Cu at (-135.8, 117.1)
- added JP23: SolderJumper_2_Open, Resistor_SMD:R_0603_1608Metric_Pad0.98x0.95mm_HandSolder, F.Cu at (-135.8, 119.6)
- added JP24: SolderJumper_2_Open, Resistor_SMD:R_0603_1608Metric_Pad0.98x0.95mm_HandSolder, F.Cu at (-135.8, 122.1)
- added JP25: SolderJumper_2_Open, Resistor_SMD:R_0603_1608Metric_Pad0.98x0.95mm_HandSolder, F.Cu at (-135.8, 124.6)
- added JP26: SolderJumper_2_Open, Resistor_SMD:R_0603_1608Metric_Pad0.98x0.95mm_HandSolder, F.Cu at (-135.8, 127.1)
- added JP27: SolderJumper_2_Open, Resistor_SMD:R_0603_1608Metric_Pad0.98x0.95mm_HandSolder, F.Cu at (-135.8, 129.7)
- added JP28: SolderJumper_2_Open, Resistor_SMD:R_0603_1608Metric_Pad0.98x0.95mm_HandSolder, F.Cu at (-135.8, 132.2)
- added JP29: SolderJumper_2_Open, Resistor_SMD:R_0603_1608Metric_Pad0.98x0.95mm_HandSolder, F.Cu at (-135.8, 134.7)
- added JP3: SolderJumper_2_Open, Jumper:SolderJumper-2_P1.3mm_Open_RoundedPad1.0x1.5mm, F.Cu at (244.8, 27.9)
- added JP30: SolderJumper_2_Open, Resistor_SMD:R_0603_1608Metric_Pad0.98x0.95mm_HandSolder, F.Cu at (-135.8, 137.2)
- added JP31: SolderJumper_2_Open, Resistor_SMD:R_0603_1608Metric_Pad0.98x0.95mm_HandSolder, F.Cu at (-135.8, 139.7)
- added JP32: SolderJumper_2_Open, Resistor_SMD:R_0603_1608Metric_Pad0.98x0.95mm_HandSolder, F.Cu at (-131.5, 109.6)
- added JP33: SolderJumper_2_Open, Resistor_SMD:R_0603_1608Metric_Pad0.98x0.95mm_HandSolder, F.Cu at (-131.5, 112.1)
- added JP34: SolderJumper_2_Open, Resistor_SMD:R_0603_1608Metric_Pad0.98x0.95mm_HandSolder, F.Cu at (-131.5, 114.6)
- added JP35: SolderJumper_2_Open, Resistor_SMD:R_0603_1608Metric_Pad0.98x0.95mm_HandSolder, F.Cu at (-131.5, 117.1)
- added JP36: SolderJumper_2_Open, Resistor_SMD:R_0603_1608Metric_Pad0.98x0.95mm_HandSolder, F.Cu at (-131.5, 119.6)
- added JP37: SolderJumper_2_Open, Resistor_SMD:R_0603_1608Metric_Pad0.98x0.95mm_HandSolder, F.Cu at (-131.5, 122.1)
- added JP38: SolderJumper_2_Open, Resistor_SMD:R_0603_1608Metric_Pad0.98x0.95mm_HandSolder, F.Cu at (-131.5, 124.6)
- added JP39: SolderJumper_2_Open, Resistor_SMD:R_0603_1608Metric_Pad0.98x0.95mm_HandSolder, F.Cu at (-131.5, 127.1)
- added JP4: SolderJumper_2_Open, Jumper:SolderJumper-2_P1.3mm_Open_RoundedPad1.0x1.5mm, F.Cu at (244.7, 25.4)
- added JP40: SolderJumper_2_Open, Resistor_SMD:R_0603_1608Metric_Pad0.98x0.95mm_HandSolder, F.Cu at (-131.5, 129.7)
- added JP41: SolderJumper_2_Open, Resistor_SMD:R_0603_1608Metric_Pad0.98x0.95mm_HandSolder, F.Cu at (-131.5, 132.2)
- added JP42: SolderJumper_2_Open, Resistor_SMD:R_0603_1608Metric_Pad0.98x0.95mm_HandSolder, F.Cu at (-131.5, 134.7)
- added JP43: SolderJumper_2_Open, Resistor_SMD:R_0603_1608Metric_Pad0.98x0.95mm_HandSolder, F.Cu at (-131.5, 137.2)
- added JP44: SolderJumper_2_Open, Resistor_SMD:R_0603_1608Metric_Pad0.98x0.95mm_HandSolder, F.Cu at (-131.5, 139.7)
- added JP45: SolderJumper_2_Open, Resistor_SMD:R_0603_1608Metric_Pad0.98x0.95mm_HandSolder, F.Cu at (-127.1, 109.6)
- added JP46: SolderJumper_2_Open, Resistor_SMD:R_0603_1608Metric_Pad0.98x0.95mm_HandSolder, F.Cu at (-127.1, 112.1)
- added JP47: SolderJumper_2_Open, Resistor_SMD:R_0603_1608Metric_Pad0.98x0.95mm_HandSolder, F.Cu at (-127.1, 114.6)
- added JP48: SolderJumper_2_Open, Resistor_SMD:R_0603_1608Metric_Pad0.98x0.95mm_HandSolder, F.Cu at (-127.1, 117.1)
- added JP49: SolderJumper_2_Open, Resistor_SMD:R_0603_1608Metric_Pad0.98x0.95mm_HandSolder, F.Cu at (-127.1, 119.6)
- added JP5: Jumper_2_Open, Connector_PinHeader_2.54mm:PinHeader_1x02_P2.54mm_Vertical, F.Cu at (144.8, 62.2)
- added JP50: SolderJumper_2_Open, Resistor_SMD:R_0603_1608Metric_Pad0.98x0.95mm_HandSolder, F.Cu at (-127.1, 122.1)
- added JP51: SolderJumper_2_Open, Resistor_SMD:R_0603_1608Metric_Pad0.98x0.95mm_HandSolder, F.Cu at (-127.1, 124.6)
- added JP52: SolderJumper_2_Open, Resistor_SMD:R_0603_1608Metric_Pad0.98x0.95mm_HandSolder, F.Cu at (-127.1, 127.1)
- added JP53: SolderJumper_2_Open, Resistor_SMD:R_0603_1608Metric_Pad0.98x0.95mm_HandSolder, F.Cu at (-127.1, 129.7)
- added JP54: SolderJumper_2_Open, Resistor_SMD:R_0603_1608Metric_Pad0.98x0.95mm_HandSolder, F.Cu at (-127.1, 132.2)
- added JP55: SolderJumper_2_Open, Resistor_SMD:R_0603_1608Metric_Pad0.98x0.95mm_HandSolder, F.Cu at (-127.1, 134.7)
- added JP56: SolderJumper_2_Open, Resistor_SMD:R_0603_1608Metric_Pad0.98x0.95mm_HandSolder, F.Cu at (-127.1, 137.2)
- added JP57: SolderJumper_2_Open, Resistor_SMD:R_0603_1608Metric_Pad0.98x0.95mm_HandSolder, F.Cu at (-127.1, 139.7)
- added JP58: SolderJumper_2_Open, Resistor_SMD:R_0603_1608Metric_Pad0.98x0.95mm_HandSolder, F.Cu at (-122.8, 109.6)
- added JP59: SolderJumper_2_Open, Resistor_SMD:R_0603_1608Metric_Pad0.98x0.95mm_HandSolder, F.Cu at (-122.8, 112.1)
- added JP6: SolderJumper_2_Open, Resistor_SMD:R_0603_1608Metric_Pad0.98x0.95mm_HandSolder, F.Cu at (-311.9, -110.7)
- added JP60: SolderJumper_2_Open, Resistor_SMD:R_0603_1608Metric_Pad0.98x0.95mm_HandSolder, F.Cu at (-122.8, 114.6)
- added JP61: SolderJumper_2_Open, Resistor_SMD:R_0603_1608Metric_Pad0.98x0.95mm_HandSolder, F.Cu at (-122.8, 117.1)
- added JP62: SolderJumper_2_Open, Resistor_SMD:R_0603_1608Metric_Pad0.98x0.95mm_HandSolder, F.Cu at (-122.8, 119.6)
- added JP63: SolderJumper_2_Open, Resistor_SMD:R_0603_1608Metric_Pad0.98x0.95mm_HandSolder, F.Cu at (-122.8, 122.1)
- added JP64: SolderJumper_2_Open, Resistor_SMD:R_0603_1608Metric_Pad0.98x0.95mm_HandSolder, F.Cu at (-122.8, 124.6)
- added JP65: SolderJumper_2_Open, Resistor_SMD:R_0603_1608Metric_Pad0.98x0.95mm_HandSolder, F.Cu at (-122.8, 127.1)
- added JP66: SolderJumper_2_Open, Resistor_SMD:R_0603_1608Metric_Pad0.98x0.95mm_HandSolder, F.Cu at (-122.8, 129.7)
- added JP67: SolderJumper_2_Open, Resistor_SMD:R_0603_1608Metric_Pad0.98x0.95mm_HandSolder, F.Cu at (-122.8, 132.2)
- added JP68: SolderJumper_2_Open, Resistor_SMD:R_0603_1608Metric_Pad0.98x0.95mm_HandSolder, F.Cu at (-122.8, 134.7)
- added JP69: SolderJumper_2_Open, Resistor_SMD:R_0603_1608Metric_Pad0.98x0.95mm_HandSolder, F.Cu at (-122.8, 137.2)
- added JP7: SolderJumper_2_Open, Resistor_SMD:R_0603_1608Metric_Pad0.98x0.95mm_HandSolder, F.Cu at (-311.4, -101.1)
- added JP70: SolderJumper_2_Open, Resistor_SMD:R_0603_1608Metric_Pad0.98x0.95mm_HandSolder, F.Cu at (-122.8, 139.7)
- added JP71: SolderJumper_2_Open, Resistor_SMD:R_0603_1608Metric_Pad0.98x0.95mm_HandSolder, F.Cu at (-118.4, 109.6)
- added JP72: SolderJumper_2_Open, Resistor_SMD:R_0603_1608Metric_Pad0.98x0.95mm_HandSolder, F.Cu at (-118.4, 112.1)
- added JP73: SolderJumper_2_Open, Resistor_SMD:R_0603_1608Metric_Pad0.98x0.95mm_HandSolder, F.Cu at (-118.4, 114.6)
- added JP74: SolderJumper_2_Open, Resistor_SMD:R_0603_1608Metric_Pad0.98x0.95mm_HandSolder, F.Cu at (-118.4, 117.1)
- added JP75: SolderJumper_2_Open, Resistor_SMD:R_0603_1608Metric_Pad0.98x0.95mm_HandSolder, F.Cu at (-118.4, 119.6)
- added JP76: SolderJumper_2_Open, Resistor_SMD:R_0603_1608Metric_Pad0.98x0.95mm_HandSolder, F.Cu at (-118.4, 122.1)
- added JP77: SolderJumper_2_Open, Resistor_SMD:R_0603_1608Metric_Pad0.98x0.95mm_HandSolder, F.Cu at (-118.4, 124.6)
- added JP78: SolderJumper_2_Open, Resistor_SMD:R_0603_1608Metric_Pad0.98x0.95mm_HandSolder, F.Cu at (-118.4, 127.1)
- added JP79: SolderJumper_2_Open, Resistor_SMD:R_0603_1608Metric_Pad0.98x0.95mm_HandSolder, F.Cu at (-118.4, 129.7)
- added JP8: SolderJumper_2_Open, Resistor_SMD:R_0603_1608Metric_Pad0.98x0.95mm_HandSolder, F.Cu at (-53.3, -139.6)
- added JP80: SolderJumper_2_Open, Resistor_SMD:R_0603_1608Metric_Pad0.98x0.95mm_HandSolder, F.Cu at (-312.0, -145.8)
- added JP81: SolderJumper_2_Open, Resistor_SMD:R_0603_1608Metric_Pad0.98x0.95mm_HandSolder, F.Cu at (-312.0, -144.3)
- added JP82: SolderJumper_2_Open, Resistor_SMD:R_0603_1608Metric_Pad0.98x0.95mm_HandSolder, F.Cu at (-312.0, -142.7)
- added JP83: SolderJumper_2_Open, Resistor_SMD:R_0603_1608Metric_Pad0.98x0.95mm_HandSolder, F.Cu at (-118.4, 139.7)
- added JP84: SolderJumper_2_Open, Resistor_SMD:R_0603_1608Metric_Pad0.98x0.95mm_HandSolder, F.Cu at (-114.1, 109.6)
- added JP85: SolderJumper_2_Open, Resistor_SMD:R_0603_1608Metric_Pad0.98x0.95mm_HandSolder, F.Cu at (-311.9, -112.8)
- added JP86: SolderJumper_2_Open, Resistor_SMD:R_0603_1608Metric_Pad0.98x0.95mm_HandSolder, F.Cu at (-114.1, 114.6)
- added JP87: SolderJumper_2_Open, Resistor_SMD:R_0603_1608Metric_Pad0.98x0.95mm_HandSolder, F.Cu at (-114.1, 117.1)
- added JP88: SolderJumper_2_Open, Resistor_SMD:R_0603_1608Metric_Pad0.98x0.95mm_HandSolder, F.Cu at (-312.0, -141.2)
- added JP89: SolderJumper_2_Open, Resistor_SMD:R_0603_1608Metric_Pad0.98x0.95mm_HandSolder, F.Cu at (-114.1, 122.1)
- added JP9: SolderJumper_2_Open, Resistor_SMD:R_0603_1608Metric_Pad0.98x0.95mm_HandSolder, F.Cu at (-53.3, -137.1)
- added JP90: SolderJumper_2_Open, Resistor_SMD:R_0603_1608Metric_Pad0.98x0.95mm_HandSolder, F.Cu at (-114.1, 124.6)
- added JP91: SolderJumper_2_Open, Resistor_SMD:R_0603_1608Metric_Pad0.98x0.95mm_HandSolder, F.Cu at (-114.1, 127.1)
- added JP92: SolderJumper_2_Open, Resistor_SMD:R_0603_1608Metric_Pad0.98x0.95mm_HandSolder, F.Cu at (-114.1, 129.7)
- added JP93: SolderJumper_2_Open, Resistor_SMD:R_0603_1608Metric_Pad0.98x0.95mm_HandSolder, F.Cu at (-114.1, 132.2)
- added JP94: SolderJumper_2_Open, Resistor_SMD:R_0603_1608Metric_Pad0.98x0.95mm_HandSolder, F.Cu at (-114.1, 134.7)
- added JP95: SolderJumper_2_Open, Resistor_SMD:R_0603_1608Metric_Pad0.98x0.95mm_HandSolder, F.Cu at (-114.1, 137.2)
- added JP96: SolderJumper_2_Open, Resistor_SMD:R_0603_1608Metric_Pad0.98x0.95mm_HandSolder, F.Cu at (-114.1, 139.7)
- added JP97: SolderJumper_2_Open, Resistor_SMD:R_0603_1608Metric_Pad0.98x0.95mm_HandSolder, F.Cu at (-109.7, 109.6)
- added JP98: SolderJumper_2_Open, Resistor_SMD:R_0603_1608Metric_Pad0.98x0.95mm_HandSolder, F.Cu at (-109.7, 112.1)
- added JP99: SolderJumper_2_Open, Resistor_SMD:R_0603_1608Metric_Pad0.98x0.95mm_HandSolder, F.Cu at (-109.7, 114.6)
- added Q1: BSS138, Package_TO_SOT_SMD:SOT-23, F.Cu at (76.8, 44.5)
- added Q11: BSS138, Package_TO_SOT_SMD:SOT-23, F.Cu at (61.5, 20.0)
- added Q2: BSS138, Package_TO_SOT_SMD:SOT-23, F.Cu at (91.5, 60.3)
- added Q3: SI2369DS-T1-GE3, Package_TO_SOT_SMD:TSOT-23, F.Cu at (247.5, 51.7)
- added Q4: BSS138, Package_TO_SOT_SMD:SOT-23, F.Cu at (79.2, 67.6)
- added Q5: BSS138, Package_TO_SOT_SMD:SOT-23, F.Cu at (48.0, 153.4)
- added Q6: BSS138, Package_TO_SOT_SMD:SOT-23, F.Cu at (70.6, 135.9)
- added R1: 1k, Resistor_SMD:R_0603_1608Metric, F.Cu at (67.5, 20.0)
- added R10: 27k, Resistor_SMD:R_0603_1608Metric, F.Cu at (240.4, 56.1)
- added R11: 10k, Resistor_SMD:R_0603_1608Metric, F.Cu at (248.0, 54.3)
- added R12: 10k, Resistor_SMD:R_0603_1608Metric, F.Cu at (247.2, 57.6)
- added R13: 20k, Resistor_SMD:R_0603_1608Metric, F.Cu at (257.3, 54.7)
- added R14: 1k, Resistor_SMD:R_0603_1608Metric, F.Cu at (191.6, 91.1)
- added R15: 1k, Resistor_SMD:R_0603_1608Metric, F.Cu at (218.2, 91.1)
- added R16: 1k, Resistor_SMD:R_0603_1608Metric, F.Cu at (26.2, 173.6)
- added R17: 1k, Resistor_SMD:R_0603_1608Metric, F.Cu at (51.8, 156.8)
- added R18: 100k, Resistor_SMD:R_0603_1608Metric, F.Cu at (51.8, 154.3)
- added R19: 190R, Resistor_SMD:R_0603_1608Metric, F.Cu at (43.3, 152.3)
- added R2: 100k, Resistor_SMD:R_0603_1608Metric, F.Cu at (64.9, 20.0)
- added R20: 1k, Resistor_SMD:R_0603_1608Metric, F.Cu at (66.8, 132.6)
- added R21: 100k, Resistor_SMD:R_0603_1608Metric, F.Cu at (66.8, 135.1)
- added R22: 1k, Resistor_SMD:R_0603_1608Metric, F.Cu at (50.3, 142.5)
- added R23: 190R, Resistor_SMD:R_0603_1608Metric, F.Cu at (75.3, 137.1)
- added R24: 1k, Resistor_SMD:R_0603_1608Metric, F.Cu at (68.3, 146.9)
- added R25: 100R, Resistor_SMD:R_0603_1608Metric, F.Cu at (70.7, 153.1)
- added R26: 100R, Resistor_SMD:R_0603_1608Metric, F.Cu at (47.9, 136.3)
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Connections:
- J1 pad 1: unconnected-(J1-Pad1) -> Net-(F1-Pad1)
- J1 pad 2: unconnected-(J1-Pad2) -> GND
- J1 pad 3: unconnected-(J1-Pad3) -> GND
- J2 pad 1: unconnected-(J2-Pin_1-Pad1) -> Net-(J2-Pin_1)
- J2 pad 2: unconnected-(J2-Pin_2-Pad2) -> Net-(J2-Pin_2)
- J3 pad 1: unconnected-(J3-Pin_1-Pad1) -> +5V
- J3 pad 2: unconnected-(J3-Pin_2-Pad2) -> /NUMPAD_VREF
- J3 pad 3: unconnected-(J3-Pin_3-Pad3) -> /NUMPAD_A_OUT
- J3 pad 4: unconnected-(J3-Pin_4-Pad4) -> GND
- J4 pad 1: unconnected-(J4-Pin_1-Pad1) -> /I2C_SCL
- J4 pad 2: unconnected-(J4-Pin_2-Pad2) -> /I2C_SDA
- J4 pad 3: unconnected-(J4-Pin_3-Pad3) -> +3V3
- J4 pad 4: unconnected-(J4-Pin_4-Pad4) -> GND
- J4 pad 5: unconnected-(J4-Pin_5-Pad5) -> /OLED_~{RES}
- J5 pad 1: unconnected-(J5-Pin_1-Pad1) -> /NSS_LISTEN
- J5 pad 2: unconnected-(J5-Pin_2-Pad2) -> /MOSI_LISTEN
- J5 pad 3: unconnected-(J5-Pin_3-Pad3) -> /MISO_LISTEN
- J5 pad 4: unconnected-(J5-Pin_4-Pad4) -> /CLK_LISTEN
- J6 pad 1: unconnected-(J6-Pin_1-Pad1) -> /NSS_LISTEN_EXTERNAL
- J6 pad 2: unconnected-(J6-Pin_2-Pad2) -> /MOSI_LISTEN_EXTERNAL
- J6 pad 3: unconnected-(J6-Pin_3-Pad3) -> /MISO_LISTEN_EXTERNAL
- J6 pad 4: unconnected-(J6-Pin_4-Pad4) -> /CLK_LISTEN_EXTERNAL
- J7 pad 1: unconnected-(J7-Pin_1-Pad1) -> GND
- J7 pad 3: unconnected-(J7-Pin_3-Pad3) -> GND
- J7 pad 4: unconnected-(J7-Pin_4-Pad4) -> /CLK_LISTEN_EXTERNAL
- J7 pad 5: unconnected-(J7-Pin_5-Pad5) -> GND
- J7 pad 6: unconnected-(J7-Pin_6-Pad6) -> /MISO_LISTEN_EXTERNAL
- J7 pad 7: unconnected-(J7-Pin_7-Pad7) -> GND
- J7 pad 8: unconnected-(J7-Pin_8-Pad8) -> /MOSI_LISTEN_EXTERNAL
- J8 pad 1: unconnected-(J8-Pin_1-Pad1) -> GND
- J8 pad 3: unconnected-(J8-Pin_3-Pad3) -> GND
- J8 pad 4: unconnected-(J8-Pin_4-Pad4) -> /CLK_LISTEN_EXTERNAL
- J8 pad 5: unconnected-(J8-Pin_5-Pad5) -> GND
- J8 pad 6: unconnected-(J8-Pin_6-Pad6) -> /MISO_LISTEN_EXTERNAL
- J8 pad 7: unconnected-(J8-Pin_7-Pad7) -> GND
- J8 pad 8: unconnected-(J8-Pin_8-Pad8) -> /MOSI_LISTEN_EXTERNAL
- J8 pad 9: unconnected-(J8-Pin_9-Pad9) -> GND
- U1 pad 11-1: unconnected-(U1-PC10-Pad11-1) -> Net-(JP80-A)
- U1 pad 11-11: unconnected-(U1-PF7-Pad11-11) -> Net-(JP61-A)
- U1 pad 11-13: unconnected-(U1-PA13-Pad11-13) -> Net-(JP19-A)
- U1 pad 11-15: unconnected-(U1-PA14-Pad11-15) -> Net-(JP20-A)
- U1 pad 11-17: unconnected-(U1-PA15-Pad11-17) -> Net-(JP21-A)
- U1 pad 11-19: unconnected-(U1-GND-Pad11-19) -> GND
- U1 pad 11-2: unconnected-(U1-PC11-Pad11-2) -> Net-(JP81-A)
- U1 pad 11-20: unconnected-(U1-GND-Pad11-20) -> GND
- U1 pad 11-21: unconnected-(U1-PB7-Pad11-21) -> Net-(JP29-A)
- U1 pad 11-22: unconnected-(U1-GND-Pad11-22) -> GND
- U1 pad 11-23: unconnected-(U1-PC13-Pad11-23) -> Net-(JP83-A)
- U1 pad 11-25: unconnected-(U1-PC14-Pad11-25) -> Net-(JP84-A)
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Routing:
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Other:
- board text added: "3V3 OK"
- board text added: "5V OK"

Commit message: main board pcb continued
Parts:
- added JP122: SolderJumper_2_Open, Resistor_SMD:R_0603_1608Metric_Pad0.98x0.95mm_HandSolder, F.Cu at (-322.6, -104.1)
- added JP123: SolderJumper_2_Open, Resistor_SMD:R_0603_1608Metric_Pad0.98x0.95mm_HandSolder, F.Cu at (-315.5, -116.8)
- added JP124: SolderJumper_2_Open, Resistor_SMD:R_0603_1608Metric_Pad0.98x0.95mm_HandSolder, F.Cu at (-315.5, -124.5)
- added JP125: SolderJumper_2_Open, Resistor_SMD:R_0603_1608Metric_Pad0.98x0.95mm_HandSolder, F.Cu at (-315.5, -127.0)
- added JP126: SolderJumper_2_Open, Resistor_SMD:R_0603_1608Metric_Pad0.98x0.95mm_HandSolder, F.Cu at (-315.5, -132.1)
- added JP127: SolderJumper_2_Open, Resistor_SMD:R_0603_1608Metric_Pad0.98x0.95mm_HandSolder, F.Cu at (-315.5, -139.7)
- added JP128: SolderJumper_2_Open, Resistor_SMD:R_0603_1608Metric_Pad0.98x0.95mm_HandSolder, F.Cu at (-178.1, 86.6)
- added JP129: SolderJumper_2_Open, Resistor_SMD:R_0603_1608Metric_Pad0.98x0.95mm_HandSolder, F.Cu at (-178.1, 89.2)
- added JP130: SolderJumper_2_Open, Resistor_SMD:R_0603_1608Metric_Pad0.98x0.95mm_HandSolder, F.Cu at (-315.5, -129.5)
- added JP131: SolderJumper_2_Open, Resistor_SMD:R_0603_1608Metric_Pad0.98x0.95mm_HandSolder, F.Cu at (-196.2, 129.6)
- added JP132: SolderJumper_2_Open, Resistor_SMD:R_0603_1608Metric_Pad0.98x0.95mm_HandSolder, F.Cu at (-322.6, -121.9)
- added JP133: SolderJumper_2_Open, Resistor_SMD:R_0603_1608Metric_Pad0.98x0.95mm_HandSolder, F.Cu at (-315.5, -121.9)
- added JP134: SolderJumper_2_Open, Resistor_SMD:R_0603_1608Metric_Pad0.98x0.95mm_HandSolder, F.Cu at (-315.5, -119.4)
- added JP135: SolderJumper_2_Open, Resistor_SMD:R_0603_1608Metric_Pad0.98x0.95mm_HandSolder, F.Cu at (-191.8, 129.6)
- added JP136: SolderJumper_2_Open, Resistor_SMD:R_0603_1608Metric_Pad0.98x0.95mm_HandSolder, F.Cu at (-191.8, 132.1)
- added JP137: SolderJumper_2_Open, Resistor_SMD:R_0603_1608Metric_Pad0.98x0.95mm_HandSolder, F.Cu at (-191.8, 134.7)
- added JP138: SolderJumper_2_Open, Resistor_SMD:R_0603_1608Metric_Pad0.98x0.95mm_HandSolder, F.Cu at (-191.8, 137.2)
- added JP139: SolderJumper_2_Open, Resistor_SMD:R_0603_1608Metric_Pad0.98x0.95mm_HandSolder, F.Cu at (-187.5, 129.6)
- added JP140: SolderJumper_2_Open, Resistor_SMD:R_0603_1608Metric_Pad0.98x0.95mm_HandSolder, F.Cu at (-315.5, -137.2)
- added JP141: SolderJumper_2_Open, Resistor_SMD:R_0603_1608Metric_Pad0.98x0.95mm_HandSolder, F.Cu at (-187.5, 134.7)
- added JP142: SolderJumper_2_Open, Resistor_SMD:R_0603_1608Metric_Pad0.98x0.95mm_HandSolder, F.Cu at (-187.5, 137.2)
- added JP67: SolderJumper_2_Open, Resistor_SMD:R_0603_1608Metric_Pad0.98x0.95mm_HandSolder, F.Cu at (-322.6, -109.2)
- added JP68: SolderJumper_2_Open, Resistor_SMD:R_0603_1608Metric_Pad0.98x0.95mm_HandSolder, F.Cu at (-322.6, -106.7)
- added JP69: SolderJumper_2_Open, Resistor_SMD:R_0603_1608Metric_Pad0.98x0.95mm_HandSolder, F.Cu at (-322.6, -137.2)
- added JP70: SolderJumper_2_Open, Resistor_SMD:R_0603_1608Metric_Pad0.98x0.95mm_HandSolder, F.Cu at (-186.8, 89.2)
- added JP71: SolderJumper_2_Open, Resistor_SMD:R_0603_1608Metric_Pad0.98x0.95mm_HandSolder, F.Cu at (-315.5, -114.3)
- added JP72: SolderJumper_2_Open, Resistor_SMD:R_0603_1608Metric_Pad0.98x0.95mm_HandSolder, F.Cu at (-315.5, -134.6)
- added TP131: TestPoint_Small, Connector_PinSocket_2.54mm:PinSocket_1x01_P2.54mm_Vertical, F.Cu at (-304.3, -109.2)
- added TP132: TestPoint_Small, Connector_PinSocket_2.54mm:PinSocket_1x01_P2.54mm_Vertical, F.Cu at (-304.3, -106.7)
- added TP133: TestPoint_Small, Connector_PinSocket_2.54mm:PinSocket_1x01_P2.54mm_Vertical, F.Cu at (-304.3, -137.2)
- added TP134: TestPoint_Small, Connector_PinSocket_2.54mm:PinSocket_1x01_P2.54mm_Vertical, F.Cu at (-186.7, 73.5)
- added TP135: TestPoint_Small, Connector_PinSocket_2.54mm:PinSocket_1x01_P2.54mm_Vertical, F.Cu at (-302.3, -114.3)
- added TP136: TestPoint_Small, Connector_PinSocket_2.54mm:PinSocket_1x01_P2.54mm_Vertical, F.Cu at (-302.3, -134.6)
- added TP185: TestPoint_Small, Connector_PinSocket_2.54mm:PinSocket_1x01_P2.54mm_Vertical, F.Cu at (-340.4, -109.2)
- added TP186: TestPoint_Small, Connector_PinSocket_2.54mm:PinSocket_1x01_P2.54mm_Vertical, F.Cu at (-340.4, -106.7)
- added TP187: TestPoint_Small, Connector_PinSocket_2.54mm:PinSocket_1x01_P2.54mm_Vertical, F.Cu at (-340.4, -137.2)
- added TP188: TestPoint_Small, Connector_PinSocket_2.54mm:PinSocket_1x01_P2.54mm_Vertical, F.Cu at (-182.1, 78.1)
- added TP189: TestPoint_Small, Connector_PinSocket_2.54mm:PinSocket_1x01_P2.54mm_Vertical, F.Cu at (-337.8, -114.3)
- added TP190: TestPoint_Small, Connector_PinSocket_2.54mm:PinSocket_1x01_P2.54mm_Vertical, F.Cu at (-337.8, -134.6)
- added TP240: TestPoint_Small, Connector_PinSocket_2.54mm:PinSocket_1x01_P2.54mm_Vertical, F.Cu at (-304.3, -104.1)
- added TP241: TestPoint_Small, Connector_PinSocket_2.54mm:PinSocket_1x01_P2.54mm_Vertical, F.Cu at (-302.3, -116.8)
- added TP242: TestPoint_Small, Connector_PinSocket_2.54mm:PinSocket_1x01_P2.54mm_Vertical, F.Cu at (-302.3, -124.5)
- added TP243: TestPoint_Small, Connector_PinSocket_2.54mm:PinSocket_1x01_P2.54mm_Vertical, F.Cu at (-302.3, -127.0)
- added TP244: TestPoint_Small, Connector_PinSocket_2.54mm:PinSocket_1x01_P2.54mm_Vertical, F.Cu at (-302.3, -132.1)
- added TP245: TestPoint_Small, Connector_PinSocket_2.54mm:PinSocket_1x01_P2.54mm_Vertical, F.Cu at (-304.3, -139.7)
- added TP246: TestPoint_Small, Connector_PinSocket_2.54mm:PinSocket_1x01_P2.54mm_Vertical, F.Cu at (-172.9, 73.5)
- added TP247: TestPoint_Small, Connector_PinSocket_2.54mm:PinSocket_1x01_P2.54mm_Vertical, F.Cu at (-172.9, 78.1)
- added TP248: TestPoint_Small, Connector_PinSocket_2.54mm:PinSocket_1x01_P2.54mm_Vertical, F.Cu at (-302.3, -129.5)
- added TP249: TestPoint_Small, Connector_PinSocket_2.54mm:PinSocket_1x01_P2.54mm_Vertical, F.Cu at (-196.0, 112.3)
- added TP250: TestPoint_Small, Connector_PinSocket_2.54mm:PinSocket_1x01_P2.54mm_Vertical, F.Cu at (-304.3, -121.9)
- added TP251: TestPoint_Small, Connector_PinSocket_2.54mm:PinSocket_1x01_P2.54mm_Vertical, F.Cu at (-302.3, -121.9)
- added TP252: TestPoint_Small, Connector_PinSocket_2.54mm:PinSocket_1x01_P2.54mm_Vertical, F.Cu at (-302.3, -119.4)
- added TP253: TestPoint_Small, Connector_PinSocket_2.54mm:PinSocket_1x01_P2.54mm_Vertical, F.Cu at (-191.4, 112.3)
- added TP254: TestPoint_Small, Connector_PinSocket_2.54mm:PinSocket_1x01_P2.54mm_Vertical, F.Cu at (-191.4, 116.9)
- added TP255: TestPoint_Small, Connector_PinSocket_2.54mm:PinSocket_1x01_P2.54mm_Vertical, F.Cu at (-191.4, 121.5)
- added TP256: TestPoint_Small, Connector_PinSocket_2.54mm:PinSocket_1x01_P2.54mm_Vertical, F.Cu at (-191.4, 126.1)
- added TP257: TestPoint_Small, Connector_PinSocket_2.54mm:PinSocket_1x01_P2.54mm_Vertical, F.Cu at (-186.8, 112.3)
- added TP258: TestPoint_Small, Connector_PinSocket_2.54mm:PinSocket_1x01_P2.54mm_Vertical, F.Cu at (-302.3, -137.2)
- added TP259: TestPoint_Small, Connector_PinSocket_2.54mm:PinSocket_1x01_P2.54mm_Vertical, F.Cu at (-186.8, 121.5)
- added TP260: TestPoint_Small, Connector_PinSocket_2.54mm:PinSocket_1x01_P2.54mm_Vertical, F.Cu at (-186.8, 126.1)
- added TP262: TestPoint_Small, Connector_PinSocket_2.54mm:PinSocket_1x01_P2.54mm_Vertical, F.Cu at (-340.4, -104.1)
- added TP263: TestPoint_Small, Connector_PinSocket_2.54mm:PinSocket_1x01_P2.54mm_Vertical, F.Cu at (-337.8, -116.8)
- added TP264: TestPoint_Small, Connector_PinSocket_2.54mm:PinSocket_1x01_P2.54mm_Vertical, F.Cu at (-337.8, -124.5)
- added TP265: TestPoint_Small, Connector_PinSocket_2.54mm:PinSocket_1x01_P2.54mm_Vertical, F.Cu at (-337.8, -127.0)
- added TP266: TestPoint_Small, Connector_PinSocket_2.54mm:PinSocket_1x01_P2.54mm_Vertical, F.Cu at (-337.8, -132.1)
- added TP267: TestPoint_Small, Connector_PinSocket_2.54mm:PinSocket_1x01_P2.54mm_Vertical, F.Cu at (-337.8, -139.7)
- added TP268: TestPoint_Small, Connector_PinSocket_2.54mm:PinSocket_1x01_P2.54mm_Vertical, F.Cu at (-163.7, 68.9)
- added TP269: TestPoint_Small, Connector_PinSocket_2.54mm:PinSocket_1x01_P2.54mm_Vertical, F.Cu at (-163.7, 73.5)
- added TP270: TestPoint_Small, Connector_PinSocket_2.54mm:PinSocket_1x01_P2.54mm_Vertical, F.Cu at (-337.8, -129.5)
- added TP271: TestPoint_Small, Connector_PinSocket_2.54mm:PinSocket_1x01_P2.54mm_Vertical, F.Cu at (-182.2, 112.3)
- added TP272: TestPoint_Small, Connector_PinSocket_2.54mm:PinSocket_1x01_P2.54mm_Vertical, F.Cu at (-340.4, -121.9)
- added TP273: TestPoint_Small, Connector_PinSocket_2.54mm:PinSocket_1x01_P2.54mm_Vertical, F.Cu at (-337.8, -121.9)
- added TP274: TestPoint_Small, Connector_PinSocket_2.54mm:PinSocket_1x01_P2.54mm_Vertical, F.Cu at (-337.8, -119.4)
- added TP275: TestPoint_Small, Connector_PinSocket_2.54mm:PinSocket_1x01_P2.54mm_Vertical, F.Cu at (-177.6, 112.3)
- added TP276: TestPoint_Small, Connector_PinSocket_2.54mm:PinSocket_1x01_P2.54mm_Vertical, F.Cu at (-177.6, 116.9)
- added TP277: TestPoint_Small, Connector_PinSocket_2.54mm:PinSocket_1x01_P2.54mm_Vertical, F.Cu at (-177.6, 121.5)
- added TP278: TestPoint_Small, Connector_PinSocket_2.54mm:PinSocket_1x01_P2.54mm_Vertical, F.Cu at (-177.6, 126.1)
- added TP279: TestPoint_Small, Connector_PinSocket_2.54mm:PinSocket_1x01_P2.54mm_Vertical, F.Cu at (-173.0, 112.3)
- added TP280: TestPoint_Small, Connector_PinSocket_2.54mm:PinSocket_1x01_P2.54mm_Vertical, F.Cu at (-337.8, -137.2)
- added TP281: TestPoint_Small, Connector_PinSocket_2.54mm:PinSocket_1x01_P2.54mm_Vertical, F.Cu at (-173.0, 121.5)
- added TP282: TestPoint_Small, Connector_PinSocket_2.54mm:PinSocket_1x01_P2.54mm_Vertical, F.Cu at (-173.0, 126.1)
- moved TP80 429.5 mm to (-340.4, -124.5)
- moved TP79 420.3 mm to (-340.4, -127.0)
- moved TP78 411.2 mm to (-340.4, -129.5)
- moved TP69 409.4 mm to (-337.8, -106.7)
- moved TP261 356.1 mm to (-340.4, -139.7)
- moved JP121 346.0 mm to (-322.6, -139.7), turned to 180 degrees
- moved TP94 338.1 mm to (-340.4, -116.8)
- moved TP230 331.1 mm to (-340.4, -132.1)
- moved TP229 328.9 mm to (-340.4, -134.6)
- moved JP32 327.8 mm to (-322.6, -116.8), turned to 180 degrees
- moved TP239 326.2 mm to (-302.3, -139.7)
- moved JP111 319.4 mm to (-322.6, -134.6)
- moved JP112 319.4 mm to (-322.6, -132.1), turned to 180 degrees
- moved JP80 315.3 mm to (-322.6, -119.4), turned to 180 degrees
- moved TP115 307.7 mm to (-335.3, -53.3)
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- renumbered C4 to C1, C20 to C10, C9 to C11, C7 to C12, C21 to C13, C1 to C3, C5 to C4, C3 to C5, C18 to C6, C6 to C7, C19 to C8, C8 to C9, D2 to D1, D11 to D10, D10 to D11, D4 to D2, D5 to D3, D3 to D4, D8 to D5, D7 to D6, D6 to D7, D1 to D8, J11 to J1, J15 to J10, J17 to J11, J5 to J12, J7 to J13, J6 to J14, J8 to J15, J1 to J2, J12 to J5, J13 to J6, J18 to J7, J2 to J8, J14 to J9, JP121 to JP1, JP13 to JP10, JP97 to JP100, JP98 to JP101, JP99 to JP102, JP100 to JP103, JP101 to JP104, JP54 to JP105, JP55 to JP106, JP56 to JP107, JP57 to JP108, JP58 to JP109, JP14 to JP11, JP59 to JP110, JP60 to JP111, JP61 to JP112, JP62 to JP113, JP63 to JP114, JP64 to JP115, JP65 to JP116, JP66 to JP117, JP67 to JP118, JP68 to JP119, JP15 to JP12, JP69 to JP120, JP118 to JP121, JP16 to JP13, JP17 to JP14, JP3 to JP143, JP5 to JP144, JP4 to JP145, JP120 to JP146, JP2 to JP147, JP1 to JP148, JP18 to JP15, JP19 to JP16, JP20 to JP17, JP21 to JP18, JP70 to JP19, JP119 to JP2, JP71 to JP20, JP72 to JP21, JP73 to JP22, JP74 to JP23, JP75 to JP24, JP76 to JP25, JP77 to JP26, JP78 to JP27, JP79 to JP28, JP80 to JP29, JP6 to JP3, JP81 to JP30, JP82 to JP31, JP83 to JP32, JP84 to JP33, JP85 to JP34, JP38 to JP35, JP39 to JP36, JP40 to JP37, JP41 to JP38, JP42 to JP39, JP7 to JP4, JP43 to JP40, JP44 to JP41, JP45 to JP42, JP46 to JP43, JP47 to JP44, JP48 to JP45, JP49 to JP46, JP50 to JP47, JP51 to JP48, JP52 to JP49, JP8 to JP5, JP53 to JP50, JP102 to JP51, JP103 to JP52, JP104 to JP53, JP105 to JP54, JP106 to JP55, JP107 to JP56, JP108 to JP57, JP109 to JP58, JP110 to JP59, JP9 to JP6, JP111 to JP60, JP112 to JP61, JP113 to JP62, JP114 to JP63, JP115 to JP64, JP116 to JP65, JP117 to JP66, JP10 to JP7, JP22 to JP73, JP23 to JP74, JP24 to JP75, JP25 to JP76, JP26 to JP77, JP27 to JP78, JP28 to JP79, JP11 to JP8, JP29 to JP80, JP30 to JP81, JP31 to JP82, JP32 to JP83, JP33 to JP84, JP34 to JP85, JP35 to JP86, JP36 to JP87, JP37 to JP88, JP86 to JP89, JP12 to JP9, JP87 to JP90, JP88 to JP91, JP89 to JP92, JP90 to JP93, JP91 to JP94, JP92 to JP95, JP93 to JP96, JP94 to JP97, JP95 to JP98, JP96 to JP99, Q11 to Q1, Q4 to Q2, Q1 to Q4, Q2 to Q5, Q5 to Q6, Q6 to Q7, R15 to R10, R14 to R11, R11 to R12, R8 to R14, R33 to R15, R5 to R16, R9 to R17, R7 to R18, R6 to R19, R34 to R20, R35 to R21, R31 to R22, R32 to R23, R16 to R24, R59 to R25, R60 to R26, R61 to R27, R62 to R28, R17 to R29, R41 to R3, R29 to R30, R18 to R31, R25 to R32, R19 to R33, R30 to R34, R24 to R35, R28 to R36, R63 to R37, R64 to R38, R22 to R39, R3 to R4, R23 to R40, R21 to R41, R26 to R42, R20 to R43, R27 to R44, R65 to R45, R66 to R46, R36 to R47, R42 to R5, R4 to R6, R43 to R7, R10 to R8, R12 to R9, SW4 to SW1, SW5 to SW2, SW6 to SW3, SW7 to SW4, SW12 to SW5, SW13 to SW6, SW14 to SW7, SW15 to SW8, TP15 to TP1, TP31 to TP10, TP96 to TP100, TP97 to TP101, TP98 to TP102, TP99 to TP103, TP100 to TP104, TP101 to TP105, TP102 to TP106, TP103 to TP107, TP104 to TP108, TP105 to TP109, TP33 to TP11, TP106 to TP110, TP107 to TP111, TP108 to TP112, TP221 to TP113, TP222 to TP114, TP223 to TP115, TP224 to TP116, TP225 to TP117, TP226 to TP118, TP227 to TP119, TP35 to TP12, TP228 to TP120, TP229 to TP121, TP230 to TP122, TP231 to TP123, TP232 to TP124, TP233 to TP125, TP234 to TP126, TP235 to TP127, TP236 to TP128, TP241 to TP129, TP37 to TP13, TP242 to TP130, TP45 to TP137, TP46 to TP138, TP47 to TP139, TP39 to TP14, TP48 to TP140, TP49 to TP141, TP50 to TP142, TP51 to TP143, TP52 to TP144, TP53 to TP145, TP54 to TP146, TP55 to TP147, TP56 to TP148, TP57 to TP149, TP41 to TP15, TP58 to TP150, TP59 to TP151, TP60 to TP152, TP173 to TP153, TP174 to TP154, TP175 to TP155, TP176 to TP156, TP177 to TP157, TP178 to TP158, TP179 to TP159, TP43 to TP16, TP180 to TP160, TP181 to TP161, TP182 to TP162, TP183 to TP163, TP184 to TP164, TP185 to TP165, TP186 to TP166, TP187 to TP167, TP188 to TP168, TP109 to TP169, TP141 to TP17, TP110 to TP170, TP111 to TP171, TP112 to TP172, TP113 to TP173, TP114 to TP174, TP115 to TP175, TP116 to TP176, TP117 to TP177, TP118 to TP178, TP119 to TP179, TP142 to TP18, TP120 to TP180, TP121 to TP181, TP122 to TP182, TP123 to TP183, TP124 to TP184, TP143 to TP19, TP61 to TP191, TP62 to TP192, TP63 to TP193, TP64 to TP194, TP65 to TP195, TP66 to TP196, TP67 to TP197, TP68 to TP198, TP69 to TP199, TP14 to TP2, TP144 to TP20, TP70 to TP200, TP71 to TP201, TP72 to TP202, TP73 to TP203, TP74 to TP204, TP75 to TP205, TP76 to TP206, TP189 to TP207, TP190 to TP208, TP191 to TP209, TP145 to TP21, TP192 to TP210, TP193 to TP211, TP194 to TP212, TP195 to TP213, TP196 to TP214, TP197 to TP215, TP198 to TP216, TP199 to TP217, TP200 to TP218, TP201 to TP219, TP146 to TP22, TP202 to TP220, TP203 to TP221, TP204 to TP222, TP125 to TP223, TP126 to TP224, TP127 to TP225, TP128 to TP226, TP129 to TP227, TP130 to TP228, TP131 to TP229, TP147 to TP23, TP132 to TP230, TP133 to TP231, TP134 to TP232, TP135 to TP233, TP136 to TP234, TP137 to TP235, TP138 to TP236, TP139 to TP237, TP140 to TP238, TP237 to TP239, TP148 to TP24, TP149 to TP25, TP150 to TP26, TP238 to TP261, TP151 to TP27, TP152 to TP28, TP6 to TP283, TP5 to TP284, TP4 to TP285, TP1 to TP286, TP7 to TP287, TP3 to TP288, TP2 to TP289, TP153 to TP29, TP17 to TP3, TP154 to TP30, TP155 to TP31, TP156 to TP32, TP77 to TP33, TP78 to TP34, TP79 to TP35, TP80 to TP36, TP81 to TP37, TP82 to TP38, TP83 to TP39, TP19 to TP4, TP84 to TP40, TP85 to TP41, TP86 to TP42, TP87 to TP43, TP88 to TP44, TP89 to TP45, TP90 to TP46, TP91 to TP47, TP92 to TP48, TP205 to TP49, TP21 to TP5, TP206 to TP50, TP207 to TP51, TP208 to TP52, TP209 to TP53, TP210 to TP54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
Connections:
- U3 pad 11-10: unconnected-(U1H-NC-Pad11-10) -> Net-(JP72-A)
- U3 pad 11-12: unconnected-(U1I-IOREF-Pad11-12) -> Net-(JP126-A)
- U3 pad 11-14: unconnected-(U1I-RESET-Pad11-14) -> Net-(JP130-A)
- U3 pad 11-16: unconnected-(U1I-3V3-Pad11-16) -> Net-(JP125-A)
- U3 pad 11-18: unconnected-(U1I-5V-Pad11-18) -> Net-(JP124-A)
- U3 pad 11-19: GND -> Net-(JP132-A)
- U3 pad 11-20: GND -> Net-(JP133-A)
- U3 pad 11-22: GND -> Net-(JP134-A)
- U3 pad 11-24: unconnected-(U1I-VIN-Pad11-24) -> Net-(JP123-A)
- U3 pad 11-26: unconnected-(U1H-NC-Pad11-26) -> Net-(JP71-A)
- U3 pad 11-29: unconnected-(U1H-PH0-Pad11-29) -> Net-(JP67-A)
- U3 pad 11-31: unconnected-(U1H-PH1-Pad11-31) -> Net-(JP68-A)
- U3 pad 11-33: unconnected-(U1I-VBAT-Pad11-33) -> Net-(JP122-A)
- U3 pad 11-49: GND -> Net-(JP139-A)
- U3 pad 11-5: unconnected-(U1I-VDD-Pad11-5) -> Net-(JP127-A)
- U3 pad 11-60: GND -> Net-(JP141-A)
- U3 pad 11-67: unconnected-(U1H-NC-Pad11-67) -> Net-(JP70-A)
- U3 pad 11-7: unconnected-(U1H-BOOT0-Pad11-7) -> Net-(JP69-A)
- U3 pad 11-8: GND -> Net-(JP140-A)
- U3 pad 12-20: GND -> Net-(JP135-A)
- U3 pad 12-32: GND -> Net-(JP131-A)
- U3 pad 12-39: GND -> Net-(JP136-A)
- U3 pad 12-54: GND -> Net-(JP137-A)
- U3 pad 12-63: GND -> Net-(JP138-A)
- U3 pad 12-7: unconnected-(U1I-AVDD-Pad12-7) -> Net-(JP129-A)
- U3 pad 12-8: unconnected-(U1I-U5V-Pad12-8) -> Net-(JP128-A)
- U3 pad 12-9: GND -> Net-(JP142-A)
Routing:
- net Net-(JP3-A): track 24.2 -> 0.00 mm
- net Net-(JP34-A): track 21.5 -> 0.00 mm
- net /PDN_UART_MOT1: track 10.4 -> 0.00 mm
- net /CLK_LISTEN: track 10.2 -> 0.00 mm
- net Net-(JP34-B): track 9.78 -> 0.00 mm
- net Net-(JP30-A): track 25.2 -> 16.2 mm
- net Net-(JP91-B): track 7.53 -> 0.00 mm
- net Net-(JP30-B): track 7.32 -> 0.00 mm
- net /MOT1_STEP: track 7.13 -> 0.00 mm
- net Net-(JP31-A): track 22.1 -> 15.8 mm
- net Net-(JP29-A): track 21.9 -> 16.1 mm
- net Net-(JP91-A): track 25.0 -> 19.7 mm

Commit message: motherboard pcb layout (MCU)
Parts:
- moved TP116 364.6 mm to (-374.4, -91.4)
- moved TP114 347.7 mm to (-374.4, -73.7)
- moved TP113 344.7 mm to (-376.9, -71.1)
- moved TP232 341.2 mm to (-374.4, -76.2)
- moved TP102 338.6 mm to (-374.4, -83.8)
- moved TP231 338.0 mm to (-374.4, -78.7)
- moved TP101 335.3 mm to (-374.4, -86.4)
- moved TP100 333.4 mm to (-376.9, -86.4)
- moved TP128 331.6 mm to (-374.4, -66.0)
- moved R22 328.9 mm to (-220.0, -143.1), turned to -90 degrees
- moved TP99 327.9 mm to (-374.4, -88.9)
- moved R23 326.2 mm to (-213.4, -140.5), turned to -90 degrees
- moved JP95 322.9 mm to (-349.4, -91.4)
- moved JP96 322.9 mm to (-349.4, -88.9), turned to 180 degrees
- moved TP214 322.7 mm to (-376.9, -88.9)
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Connections:
- R22 pad 2: /I2C_SCL -> Net-(JP81-A)
- R23 pad 2: /I2C_SDA -> Net-(JP82-A)
Routing:
- net Net-(JP91-A): track 19.7 -> 0.00 mm
- net Net-(JP30-A): track 16.2 -> 0.00 mm
- net Net-(JP29-A): track 16.1 -> 0.00 mm
- net Net-(JP31-A): track 15.8 -> 0.00 mm
Other:
- board text added: "τ"
