File: KiCad/motherboard/motherboard.kicad_sch (KiCad schematic)
At the start: 558 parts, among them J1 Conn_01x06_Pin, J10 Conn_01x04_Pin, J11 DB25_Socket_MountingHoles, J12 Conn_01x04_Pin, J13 1761681-9, J14 Conn_01x04_Pin, J15 1761681-9, J2 Barrel_Jack_Switch, J3 Conn_01x04_Pin, J4 Conn_01x05_Pin, J5 Conn_01x06_Pin, J6 Conn_01x04_Pin, J7 Conn_01x09_Pin, J8 Conn_01x02_Socket, J9 Conn_01x04_Pin, Q1 BSS138, Q2 BSS138, Q3 SI2369DS-T1-GE3, Q4 BSS138, Q5 BSS138, Q6 BSS138, Q7 BSS138, SW1 EmergencyStop, SW2 TiltSwitch, SW3 DoorSwitch, SW4 AdditionalSlot, SW5 SW_Push, SW6 SW_Push, SW7 SW_Push, SW8 SW_Push, U1 P7803B-1000, U10 24LC512, U2 P7805B-1000, U4 ASSR-1218, U5 TMC2209, U6 TMC2209, U7 LSF0204QPWRQ1, U8 LTV-817S, U9 LTV-817S

Commit message: exports
Other:
- title: Motherboard -> K.I.T.T.E.N. Alaplap
Changed lines of the file:
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@@
 	(paper "A2")
 	(title_block
-		(title "Motherboard")
+		(title "K.I.T.T.E.N. Alaplap")
 		(date "2025-11-17")
 		(rev "1.0")

Commit message: ppt continued
Other:
- note added: "ENCODER 2"
Changed lines of the file:
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@@
 		)
 	)
-	(text "ENCODER 1"
+	(text "ENCODER 2"
 		(exclude_from_sim no)
 		(at 75.565 206.375 0)
