File: KiCad/buttons/buttons.kicad_sch (KiCad schematic)
At the start: 29 parts, among them J8 Conn_01x09_Pin, SW1 Cherry Switch Single, SW2 Cherry Switch Single, SW4 Cherry Switch Single, SW5 Cherry Switch Single, SW6 Cherry Switch Single, SW7 Cherry Switch Single, SW8 Cherry Switch Single

Commit message: schematics finished
Connections:
- net BTN_ADDITIONAL renamed BTN_EXTERNAL_EXTRA
Other:
- note added: "Csatlakozó"
- note added: "GOMBOK"
- note added: "U_{H} = 3.3· 10/11 = 3V T_{charge} = 0.1ms -> 5T = 0.5ms T_{discharge} = 1ms -> 5T = 5ms"
- note removed: "U_{H} = 3.3· 10/11 = 3V Tau_{charge} = 0.1ms -> 5Tau = 0.5ms Tau_{discharge} = 1ms -> 5Tau = 5ms"
- moved on the sheet: C7, J8, R11, R12, SW7

Commit message: PCB designs started
Parts:
- added H1, H2, H3, H4: MountingHole, MountingHole:MountingHole_3.2mm_M3, symbol Mechanical:MountingHole
- renumbered C6 to C1, C4 to C2, C1 to C3, C8 to C4, C3 to C5, C5 to C6, J8 to J1, R9 to R1, R14 to R10, R6 to R11, R8 to R12, R11 to R13, R12 to R14, R22 to R2, R1 to R3, R10 to R4, R23 to R5, R2 to R6, R13 to R7, R5 to R8, R7 to R9, SW6 to SW1, SW1 to SW2, SW2 to SW3, SW8 to SW4, SW4 to SW5, SW5 to SW6
Connections:
- net BTN_FIX_AX: now also J1.3 (Pin_3); no longer J1.2 (Pin_2)
- net BTN_MEMSLOT: now also J1.2 (Pin_2); no longer J1.4 (Pin_4)
- net BTN_SET: now also J1.4 (Pin_4); no longer J1.6 (Pin_6)
- net BTN_TRACKED_AX: now also J1.6 (Pin_6); no longer J1.3 (Pin_3)
Other:
- note added: "Rögzítőfuratok"
- moved on the sheet: C1, C2, C3, C4, C5, C6, C7, R1, R10, R11, R12, R13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

Commit message: PPT
Other:
- title: (none) -> Buttons
Changed lines of the file:
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@@
 	(generator_version "9.0")
 	(paper "A4")
+	(title_block
+		(title "Buttons")
+		(date "2025-11-17")
+		(rev "1.0")
+	)
 	(rectangle
 		(start 178.435 97.663)

Commit message: exports
Other:
- title: Buttons -> Gomb panel
Changed lines of the file:
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@@
 	(paper "A4")
 	(title_block
-		(title "Buttons")
+		(title "Gomb panel")
 		(date "2025-11-17")
 		(rev "1.0")
